Commit message: Working gazibo and rviz

File: ws/src/mserve_description/urdf/mserve_core.xacro (robot description, xacro)
@@ -10,7 +10,8 @@
      <!-- Wheel Properties (in meteres)  -->
   <xacro:property name="wheel_radius" value="0.05"/>
-  <xacro:property name="wheel_length" value="0.04"/>
+  <xacro:property name="wheel_width" value="0.04"/>
   <xacro:property name="wheel_mass" value="0.765"/>
-  <xacro:property name="wheel_y_offset" value="0.18"/>
+  <xacro:property name="wheel_spacing" value="0.015"/>
+  <xacro:property name="wheel_y_offset" value="${(chassis_width / 2.0 ) + wheel_spacing + (wheel_width / 2)}"/>
   <xacro:property name="wheel_no_load_rpm" value="200.0"/>
   <xacro:property name="wheel_rated_rpm" value="115.0"/>
@@ -30,13 +31,15 @@
   <xacro:property name="caster_radius" value="0.05"/>
   <xacro:property name="caster_mass" value="0.3"/>
-  <xacro:property name="caster_x" value="0.30"/>
+  <xacro:property name="caster_offset" value="0.00"/>
+  <xacro:property name="caster_x" value="${(chassis_length - caster_radius - caster_offset)}"/>
   <xacro:property name="caster_z" value="0"/>
   <!-- Lidar Properties (in meteres, kG) -->
   <xacro:property name="lidar_radius" value="0.04"/>
   <xacro:property name="lidar_length" value="0.04"/>
-  <xacro:property name="lidar_mass" value="0.2"/>
-  <xacro:property name="lidar_x" value="0.24"/>
+  <xacro:property name="lidar_mass" value="0.1"/>
+  <xacro:property name="lidar_offset" value="0.00"/>
+  <xacro:property name="lidar_x" value="${chassis_length / 2.0 + lidar_offset}"/>
   <xacro:property name="lidar_y" value="0.0"/>
-  <xacro:property name="lidar_z" value="0.19"/>
+  <xacro:property name="lidar_z" value="${chassis_height + lidar_length / 2.0}"/>
   <!-- Camera Properties (in meteres, kG) -->
   <xacro:property name="camera_depth" value="0.05"/>
@@ -44,7 +47,8 @@
   <xacro:property name="camera_height" value="0.04"/>
   <xacro:property name="camera_mass" value="0.15"/>
-  <xacro:property name="camera_x" value="0.32"/>
+  <xacro:property name="camera_offset" value="0.01"/>
+  <xacro:property name="camera_x" value="${chassis_length - (camera_depth / 2) - camera_offset}"/>
   <xacro:property name="camera_y" value="0.0"/>
-  <xacro:property name="camera_z" value="0.14"/>
+  <xacro:property name="camera_z" value="${chassis_height + camera_height / 2.0}"/>
   <!-- Display Properties (in meteres)  -->
   <xacro:property name="display_width" value="0.12"/>
@@ -52,14 +56,16 @@
   <xacro:property name="display_height" value="0.08"/>
   <xacro:property name="display_mass" value="0.25"/>
+  <xacro:property name="display_offset" value="0.05"/>
   <xacro:property name="display_x" value="${chassis_length + display_depth / 2.0}"/>
   <xacro:property name="display_y" value="0.0"/>
-  <xacro:property name="display_z" value="${chassis_height * 0.65}"/>
+  <xacro:property name="display_z" value="${display_height / 2.0 + display_offset}"/>
   <!-- Arm Mount Properties (in meteres, kG) -->
   <xacro:property name="arm_mount_radius" value="0.03"/>
   <xacro:property name="arm_mount_length" value="0.06"/>
   <xacro:property name="arm_mount_mass" value="0.4"/>
-  <xacro:property name="arm_mount_x" value="0.08"/>
+  <xacro:property name="arm_mount_offset" value="0.05"/>
+  <xacro:property name="arm_mount_x" value="${arm_mount_offset}"/>
   <xacro:property name="arm_mount_y" value="0.0"/>
-  <xacro:property name="arm_mount_z" value="0.20"/>
+  <xacro:property name="arm_mount_z" value="${chassis_height + arm_mount_length / 2.0}"/>
   <!-- Aggregate values used by Gazebo drive systems -->
   <xacro:property name="robot_total_mass" value="${chassis_mass + 2.0 * wheel_mass + caster_mass + lidar_mass + camera_mass + display_mass + arm_mount_mass}"/>
@@ -119,5 +125,5 @@
     <visual>
       <geometry>
-        <cylinder radius="${wheel_radius}" length="${wheel_length}"/>
+        <cylinder radius="${wheel_radius}" length="${wheel_width}"/>
       </geometry>
       <material name="wheel_black"/>
@@ -125,5 +131,5 @@
     <collision>
       <geometry>
-        <cylinder radius="${wheel_radius}" length="${wheel_length}"/>
+        <cylinder radius="${wheel_radius}" length="${wheel_width}"/>
       </geometry>
     </collision>
@@ -131,5 +137,5 @@
       mass="${wheel_mass}"
       radius="${wheel_radius}"
-      length="${wheel_length}"
+      length="${wheel_width}"
       origin_xyz="0 0 0"
       origin_rpy="0 0 0"/>
@@ -147,5 +153,5 @@
     <visual>
       <geometry>
-        <cylinder radius="${wheel_radius}" length="${wheel_length}"/>
+        <cylinder radius="${wheel_radius}" length="${wheel_width}"/>
       </geometry>
       <material name="wheel_black"/>
@@ -153,5 +159,5 @@
     <collision>
       <geometry>
-        <cylinder radius="${wheel_radius}" length="${wheel_length}"/>
+        <cylinder radius="${wheel_radius}" length="${wheel_width}"/>
       </geometry>
     </collision>
@@ -159,5 +165,5 @@
       mass="${wheel_mass}"
       radius="${wheel_radius}"
-      length="${wheel_length}"
+      length="${wheel_width}"
       origin_xyz="0 0 0"
       origin_rpy="0 0 0"/>
