Commit message: Wire up Nav2 and fix real-hardware doorway navigation
Switches localization to AMCL + map_server (mserve_nav2.launch.py,
nav2_params.yaml), adds the --nav2 flag to run_stack.sh, and fixes a
lifecycle_manager bug where a genuine BT bringup FAILURE was logged and
treated as success (surfaced by slam_toolbox blocking its executor on a
slow pose-graph load past the old 2s service timeout).

On real hardware the robot then stalled at interior doorways. Root causes
tracked down by measuring the actual doorway from the saved map and the
real chassis: robot_radius was a circle sized to the chassis diagonal,
penalizing every heading by the full diagonal even driving straight
through — replaced with a measured rectangular footprint on both
costmaps, freeing up enough real margin to also fix inflation_radius
(0.4 blocked doorways outright; overcorrecting to 0.1 left NavFn with no
cost gradient toward corridor centerlines, so paths hugged one wall).
Settled at 0.15. mserve_core.xacro's chassis_width also corrected to the
measured value.

Co-Authored-By: Claude Sonnet 5 <noreply@anthropic.com>

File: ws/src/mserve_description/urdf/mserve_core.xacro (robot description, xacro)
@@ -3,17 +3,20 @@
   <xacro:include filename="inertial_macros.xacro"/>
     <!-- Chassis Properties (in meteres, kG) -->
-  <xacro:property name="chassis_length" value="0.37"/>
-  <xacro:property name="chassis_width" value="0.25"/>
+  <xacro:property name="chassis_length" value="0.37"/>  <!-- measured 2026-07-19 -->
+  <xacro:property name="chassis_width" value="0.20"/>  <!-- measured 2026-07-19: body width, excludes wheels -->
   <xacro:property name="chassis_height" value="0.15"/>
   <xacro:property name="chassis_mass" value="12.0"/>
   <!-- Measured 2026-07-19: 75mm from the wheel axis (base_link origin — the
        wheel joints below attach directly to base_link) to the back of the
-       frame. chassis_length/chassis_width/chassis_height remain rough
-       placeholders — the real chassis is an open aluminum-extrusion rail
-       frame, not a solid box, and camera/lidar heights are measured
-       directly from the wheel axis (see mserve_lidar.xacro/
-       mserve_camera.xacro) rather than through chassis_height, so that
-       placeholder mostly just affects this visual box's own proportions
-       now, not sensor placement. -->
+       frame, and chassis_length/chassis_width are now real measurements
+       (370x200mm body). chassis_height remains a rough placeholder — the
+       real chassis is an open aluminum-extrusion rail frame, not a solid
+       box, and camera/lidar heights are measured directly from the wheel
+       axis (see mserve_lidar.xacro/mserve_camera.xacro) rather than through
+       chassis_height, so that placeholder mostly just affects this visual
+       box's own proportions now, not sensor placement. Nav2's footprint
+       (ws/src/interfaces/config/nav2_params.yaml) uses the 315mm
+       wheel-to-wheel outer width directly, not chassis_width here, since
+       collision avoidance needs the true outer envelope including wheels. -->
   <xacro:property name="chassis_joint_x" value="-0.075"/>
      <!-- Wheel Properties (in meteres)  -->
