Commit message: Controlable in gazibo using keyboard

File: ws/src/mserve_description/urdf/mserve.urdf.xacro (robot description, xacro)
@@ -3,3 +3,5 @@
   <!-- Include the core robot definition -->
   <xacro:include filename="mserve_core.xacro"/>
+  <!-- Include Gazebo-specific simulation tuning -->
+  <xacro:include filename="mserve_gazebo.xacro"/>
 </robot>

File: ws/src/mserve_description/urdf/mserve_core.xacro (robot description, xacro)
@@ -9,13 +9,27 @@
   <xacro:property name="chassis_joint_x" value="-0.10"/>
      <!-- Wheel Properties (in meteres)  -->
-  <xacro:property name="wheel_radius" value="0.1"/>
+  <xacro:property name="wheel_radius" value="0.05"/>
   <xacro:property name="wheel_length" value="0.04"/>
   <xacro:property name="wheel_mass" value="0.765"/>
   <xacro:property name="wheel_y_offset" value="0.18"/>
+  <xacro:property name="wheel_no_load_rpm" value="200.0"/>
+  <xacro:property name="wheel_rated_rpm" value="115.0"/>
+  <xacro:property name="wheel_rated_torque" value="0.96"/>
+  <xacro:property name="wheel_stall_torque" value="2.0"/>
+  <xacro:property name="wheel_torque_constant" value="0.75"/>
+  <xacro:property name="wheel_speed_constant_rpm_per_volt" value="11.1"/>
+  <xacro:property name="wheel_encoder_resolution" value="4096"/>
+  <xacro:property name="wheel_single_wheel_load" value="10.0"/>
+  <xacro:property name="wheel_separation" value="${2.0 * wheel_y_offset}"/>
+  <xacro:property name="wheel_velocity_limit" value="${wheel_no_load_rpm * 2.0 * pi / 60.0}"/>
+  <xacro:property name="wheel_rated_velocity" value="${wheel_rated_rpm * 2.0 * pi / 60.0}"/>
+  <xacro:property name="wheel_effort_limit" value="${wheel_stall_torque}"/>
+  <xacro:property name="wheel_joint_damping" value="0.05"/>
+  <xacro:property name="wheel_joint_friction" value="0.02"/>
   <!-- Caster Properties (in meteres)  -->
   <xacro:property name="caster_radius" value="0.05"/>
   <xacro:property name="caster_mass" value="0.3"/>
   <xacro:property name="caster_x" value="0.30"/>
-  <xacro:property name="caster_z" value="-0.01"/>
+  <xacro:property name="caster_z" value="0"/>
   <!-- Lidar Properties (in meteres, kG) -->
   <xacro:property name="lidar_radius" value="0.04"/>
@@ -48,4 +62,6 @@
   <xacro:property name="arm_mount_y" value="0.0"/>
   <xacro:property name="arm_mount_z" value="0.20"/>
+  <!-- Aggregate values used by Gazebo drive systems -->
+  <xacro:property name="robot_total_mass" value="${chassis_mass + 2.0 * wheel_mass + caster_mass + lidar_mass + camera_mass + display_mass + arm_mount_mass}"/>
   <!-- Materials -->
   <material name="chassis_blue">
@@ -97,4 +113,6 @@
     <origin xyz="0 ${wheel_y_offset} 0" rpy="${-pi / 2.0} 0 0"/>
     <axis xyz="0 0 1"/>
+    <limit effort="${wheel_effort_limit}" velocity="${wheel_velocity_limit}"/>
+    <dynamics damping="${wheel_joint_damping}" friction="${wheel_joint_friction}"/>
   </joint>
   <link name="left_wheel">
@@ -123,4 +141,6 @@
     <origin xyz="0 ${-wheel_y_offset} 0" rpy="${pi / 2.0} 0 0"/>
     <axis xyz="0 0 -1"/>
+    <limit effort="${wheel_effort_limit}" velocity="${wheel_velocity_limit}"/>
+    <dynamics damping="${wheel_joint_damping}" friction="${wheel_joint_friction}"/>
   </joint>
   <link name="right_wheel">

Commit message: Added lidar to simulation

File: ws/src/mserve_description/urdf/mserve.urdf.xacro (robot description, xacro)
@@ -3,4 +3,7 @@
   <!-- Include the core robot definition -->
   <xacro:include filename="mserve_core.xacro"/>
+  <!-- Include Lidar -->
+  <xacro:include filename="mserve_lidar.xacro"/>
+  <xacro:mserve_lidar parent_link="chassis"/>
   <!-- Include Gazebo-specific simulation tuning -->
   <xacro:include filename="mserve_gazebo.xacro"/>

File: ws/src/mserve_description/urdf/mserve_core.xacro (robot description, xacro)
@@ -34,12 +34,4 @@
   <xacro:property name="caster_x" value="${(chassis_length - caster_radius - caster_offset)}"/>
   <xacro:property name="caster_z" value="0"/>
-  <!-- Lidar Properties (in meteres, kG) -->
-  <xacro:property name="lidar_radius" value="0.04"/>
-  <xacro:property name="lidar_length" value="0.04"/>
-  <xacro:property name="lidar_mass" value="0.1"/>
-  <xacro:property name="lidar_offset" value="0.00"/>
-  <xacro:property name="lidar_x" value="${chassis_length / 2.0 + lidar_offset}"/>
-  <xacro:property name="lidar_y" value="0.0"/>
-  <xacro:property name="lidar_z" value="${chassis_height + lidar_length / 2.0}"/>
   <!-- Camera Properties (in meteres, kG) -->
   <xacro:property name="camera_depth" value="0.05"/>
@@ -68,6 +60,4 @@
   <xacro:property name="arm_mount_y" value="0.0"/>
   <xacro:property name="arm_mount_z" value="${chassis_height + arm_mount_length / 2.0}"/>
-  <!-- Aggregate values used by Gazebo drive systems -->
-  <xacro:property name="robot_total_mass" value="${chassis_mass + 2.0 * wheel_mass + caster_mass + lidar_mass + camera_mass + display_mass + arm_mount_mass}"/>
   <!-- Materials -->
   <material name="chassis_blue">
@@ -80,7 +70,4 @@
     <color rgba="0.15 0.15 0.15 1.0"/>
   </material>
-  <material name="sensor_green">
-    <color rgba="0.27 0.67 0.47 1.0"/>
-  </material>
   <!-- BASE LINK -->
   <link name="base_link"/>
@@ -193,29 +180,4 @@
       origin_rpy="0 0 0"/>
   </link>
-  <!-- LIDAR JOINT -->
-  <joint name="lidar_joint" type="fixed">
-    <parent link="chassis"/>
-    <child link="lidar_link"/>
-    <origin xyz="${lidar_x} ${lidar_y} ${lidar_z}" rpy="0 0 0"/>
-  </joint>
-  <link name="lidar_link">
-    <visual>
-      <geometry>
-        <cylinder radius="${lidar_radius}" length="${lidar_length}"/>
-      </geometry>
-      <material name="sensor_green"/>
-    </visual>
-    <collision>
-      <geometry>
-        <cylinder radius="${lidar_radius}" length="${lidar_length}"/>
-      </geometry>
-    </collision>
-    <xacro:inertial_cylinder
-      mass="${lidar_mass}"
-      radius="${lidar_radius}"
-      length="${lidar_length}"
-      origin_xyz="0 0 0"
-      origin_rpy="0 0 0"/>
-  </link>
   <!-- CAMERA JOINT -->
   <joint name="camera_joint" type="fixed">

File: ws/src/mserve_description/urdf/mserve_gazebo.xacro (robot description, xacro)
@@ -8,4 +8,5 @@
   <xacro:property name="diff_drive_child_frame_id" value="base_link"/>
   <xacro:property name="diff_drive_odom_publish_frequency" value="50.0"/>
+  <xacro:property name="robot_total_mass" value="${chassis_mass + 2.0 * wheel_mass + caster_mass + lidar_riser_mass + lidar_mass + camera_mass + display_mass + arm_mount_mass}"/>
   <xacro:property name="diff_drive_max_linear_velocity" value="${wheel_rated_velocity * wheel_radius}"/>
   <xacro:property name="diff_drive_max_angular_velocity" value="${2.0 * diff_drive_max_linear_velocity / wheel_separation}"/>

Commit message: Camera Added + updated models

File: ws/src/mserve_description/urdf/mserve.urdf.xacro (robot description, xacro)
@@ -3,4 +3,7 @@
   <!-- Include the core robot definition -->
   <xacro:include filename="mserve_core.xacro"/>
+  <!-- Include Camera -->
+  <xacro:include filename="mserve_camera.xacro"/>
+  <xacro:mserve_camera parent_link="chassis"/>
   <!-- Include Lidar -->
   <xacro:include filename="mserve_lidar.xacro"/>

File: ws/src/mserve_description/urdf/mserve_core.xacro (robot description, xacro)
@@ -34,13 +34,4 @@
   <xacro:property name="caster_x" value="${(chassis_length - caster_radius - caster_offset)}"/>
   <xacro:property name="caster_z" value="0"/>
-  <!-- Camera Properties (in meteres, kG) -->
-  <xacro:property name="camera_depth" value="0.05"/>
-  <xacro:property name="camera_width" value="0.08"/>
-  <xacro:property name="camera_height" value="0.04"/>
-  <xacro:property name="camera_mass" value="0.15"/>
-  <xacro:property name="camera_offset" value="0.01"/>
-  <xacro:property name="camera_x" value="${chassis_length - (camera_depth / 2) - camera_offset}"/>
-  <xacro:property name="camera_y" value="0.0"/>
-  <xacro:property name="camera_z" value="${chassis_height + camera_height / 2.0}"/>
   <!-- Display Properties (in meteres)  -->
   <xacro:property name="display_width" value="0.12"/>
@@ -180,30 +171,4 @@
       origin_rpy="0 0 0"/>
   </link>
-  <!-- CAMERA JOINT -->
-  <joint name="camera_joint" type="fixed">
-    <parent link="chassis"/>
-    <child link="camera_link"/>
-    <origin xyz="${camera_x} ${camera_y} ${camera_z}" rpy="0 0 0"/>
-  </joint>
-  <link name="camera_link">
-    <visual>
-      <geometry>
-        <box size="${camera_depth} ${camera_width} ${camera_height}"/>
-      </geometry>
-      <material name="trim_grey"/>
-    </visual>
-    <collision>
-      <geometry>
-        <box size="${camera_depth} ${camera_width} ${camera_height}"/>
-      </geometry>
-    </collision>
-    <xacro:inertial_box
-      mass="${camera_mass}"
-      x="${camera_depth}"
-      y="${camera_width}"
-      z="${camera_height}"
-      origin_xyz="0 0 0"
-      origin_rpy="0 0 0"/>
-  </link>
   <!-- DISPLAY JOINT -->
   <joint name="display_joint" type="fixed">
