Commit message: Real chassis/sensor dimensions, camera fix, defined-cycle capture loops
Robot dimensions (mserve_description, mserve_params.yaml): wheel
separation (350->305mm) and radius (80->50.35mm) replaced with physical
measurements — the old wheel_radius was ~59% off, meaning real speed and
odometry have both been wrong until now. Lidar/camera positions now
measured directly from the wheel axis (base_link origin) rather than
derived through chassis_height, which was never a real measurement and
already inconsistent with the camera's actual mount height. Camera model
switched from mserve_depth_camera.xacro back to the plain mserve_camera.xacro
— the real hardware is a USB webcam (v4l2_camera), not RGBD; flipped
test_urdf_load.py's assertion back to match.

Camera/lidar reliability (mserve_camera, mserve_lidar): both capture loops
now run on a defined cycle (capture_rate_hz/scan_rate_hz) instead of
trusting the underlying blocking hardware call to self-rate-limit. Root
cause of a real incident: mserve_camera hit a sustained V4L2 "No such
device" error with no dmesg evidence of an actual USB disconnect, and
without independent pacing that produced 14M+ log lines and pinned a full
CPU core within minutes — severe enough that ros2 launch's own stdout
multiplexing spiked system-wide CPU past 90%. mserve_lidar had the
identical unbounded-retry pattern, fixed the same way. Both log a
rate-limited health summary during sustained failure instead of either
silent spinning or per-failure spam.

Camera CPU (mserve_camera): compressed/raw image encoding is now gated on
actual subscriber count, not just lifecycle-active state — in normal
operation nothing subscribes to camera/image_raw/compressed (both web UI
pages stream image_raw directly), so the full JPEG encode was running
every frame for zero consumers. Measured idle CPU drop: ~40-60% to ~1.7%.
Headroom recovery ahead of Nav2.

Co-Authored-By: Claude Sonnet 5 <noreply@anthropic.com>

File: ws/src/mserve_description/urdf/mserve.urdf.xacro (robot description, xacro)
@@ -3,10 +3,9 @@
   <!-- Include the core robot definition -->
   <xacro:include filename="mserve_core.xacro"/>
-  <!-- Pi Camera (disabled — replaced by depth camera below) -->
-  <!-- <xacro:include filename="mserve_camera.xacro"/> -->
-  <!-- <xacro:mserve_camera parent_link="chassis"/> -->
-  <!-- Depth Camera -->
-  <xacro:include filename="mserve_depth_camera.xacro"/>
-  <xacro:mserve_depth_camera parent_link="chassis"/>
+  <!-- USB webcam (mserve_camera wraps v4l2_camera) — plain RGB, not depth.
+       mserve_depth_camera.xacro (kept in the tree, just unused) modeled an
+       RGBD camera that doesn't match this hardware — confirmed 2026-07-19. -->
+  <xacro:include filename="mserve_camera.xacro"/>
+  <xacro:mserve_camera parent_link="chassis"/>
   <!-- Include Lidar -->
   <xacro:include filename="mserve_lidar.xacro"/>

File: ws/src/mserve_description/urdf/mserve_camera.xacro (robot description, xacro)
@@ -2,14 +2,24 @@
 <robot xmlns:xacro="http://www.ros.org/wiki/xacro">
   <xacro:include filename="inertial_macros.xacro"/>
-  <!-- Raspberry Pi Camera Module 3 style defaults. Keep these isolated so a
-       later hardware swap only needs this file updated. -->
+  <!-- USB webcam (not a CSI Pi Camera Module — mserve_camera wraps
+       v4l2_camera). width/height measured 2026-07-19: 80x30mm. camera_depth
+       is still the old Pi Camera Module 3 placeholder (11.5mm) — no real
+       depth measurement yet, and it barely matters visually next to the
+       80x30 footprint. -->
   <xacro:property name="camera_depth" value="0.0115"/>
-  <xacro:property name="camera_width" value="0.025"/>
-  <xacro:property name="camera_height" value="0.024"/>
+  <xacro:property name="camera_width" value="0.080"/>
+  <xacro:property name="camera_height" value="0.030"/>
   <xacro:property name="camera_mass" value="0.005"/>
-  <xacro:property name="camera_offset" value="0.005"/>
-  <xacro:property name="camera_x" value="${chassis_length + camera_depth / 2.0 + camera_offset}"/>
+  <!-- Measured 2026-07-19, both from the wheel axis (base_link origin):
+       280mm forward, 115mm up. camera_x is chassis-local (this macro's
+       parent_link is "chassis" — see mserve_core.xacro's chassis_joint_x
+       comment), so it's the wheel-axis measurement minus chassis_joint_x.
+       camera_z is direct — no chassis_height in this calculation, the real
+       chassis is an open rail frame, not a solid box (same reasoning as
+       mserve_lidar.xacro). -->
+  <xacro:property name="camera_x_from_wheel_axis" value="0.280"/>
+  <xacro:property name="camera_x" value="${camera_x_from_wheel_axis - chassis_joint_x}"/>
   <xacro:property name="camera_y" value="0.0"/>
-  <xacro:property name="camera_z" value="${chassis_height + camera_height / 2.0}"/>
+  <xacro:property name="camera_z" value="0.115"/>
   <xacro:property name="camera_image_topic" value="camera/image_raw"/>
   <xacro:property name="camera_info_topic" value="camera/camera_info"/>

File: ws/src/mserve_description/urdf/mserve_core.xacro (robot description, xacro)
@@ -7,11 +7,26 @@
   <xacro:property name="chassis_height" value="0.15"/>
   <xacro:property name="chassis_mass" value="12.0"/>
-  <xacro:property name="chassis_joint_x" value="-0.10"/>
+  <!-- Measured 2026-07-19: 75mm from the wheel axis (base_link origin — the
+       wheel joints below attach directly to base_link) to the back of the
+       frame. chassis_length/chassis_width/chassis_height remain rough
+       placeholders — the real chassis is an open aluminum-extrusion rail
+       frame, not a solid box, and camera/lidar heights are measured
+       directly from the wheel axis (see mserve_lidar.xacro/
+       mserve_camera.xacro) rather than through chassis_height, so that
+       placeholder mostly just affects this visual box's own proportions
+       now, not sensor placement. -->
+  <xacro:property name="chassis_joint_x" value="-0.075"/>
      <!-- Wheel Properties (in meteres)  -->
-  <xacro:property name="wheel_radius" value="0.05"/>
+  <xacro:property name="wheel_radius" value="0.05035"/>  <!-- measured 2026-07-19: 100.7mm diameter -->
   <xacro:property name="wheel_width" value="0.04"/>
   <xacro:property name="wheel_mass" value="0.765"/>
-  <xacro:property name="wheel_spacing" value="0.015"/>
-  <xacro:property name="wheel_y_offset" value="${(chassis_width / 2.0 ) + wheel_spacing + (wheel_width / 2)}"/>
+  <!-- Measured 2026-07-19 (real robot, matches mserve_params.yaml's
+       mserve_base.limits.wheel_separation — keep both in sync). Drives
+       wheel_y_offset directly rather than the other way around, since this
+       is now a real measurement and chassis_width is still a guess — a
+       kinematically-critical dimension shouldn't be derived from an
+       unmeasured cosmetic one. -->
+  <xacro:property name="wheel_separation" value="0.305"/>
+  <xacro:property name="wheel_y_offset" value="${wheel_separation / 2.0}"/>
   <xacro:property name="wheel_no_load_rpm" value="200.0"/>
   <xacro:property name="wheel_rated_rpm" value="115.0"/>
@@ -22,5 +37,4 @@
   <xacro:property name="wheel_encoder_resolution" value="4096"/>
   <xacro:property name="wheel_single_wheel_load" value="10.0"/>
-  <xacro:property name="wheel_separation" value="${2.0 * wheel_y_offset}"/>
   <xacro:property name="wheel_velocity_limit" value="${wheel_no_load_rpm * 2.0 * pi / 60.0}"/>
   <xacro:property name="wheel_rated_velocity" value="${wheel_rated_rpm * 2.0 * pi / 60.0}"/>

File: ws/src/mserve_description/urdf/mserve_depth_camera.xacro (robot description, xacro)
@@ -26,7 +26,18 @@
   <xacro:property name="camera_mass"         value="0.072"/>  <!-- named camera_mass for mserve_gazebo.xacro total mass -->
   <xacro:property name="depth_camera_offset" value="0.005"/>
-  <!-- Mount flush with the front face of the chassis, at chassis-top height -->
-  <xacro:property name="depth_camera_x" value="${chassis_length + depth_camera_depth / 2.0 + depth_camera_offset}"/>
+  <!-- Measured 2026-07-19: 280mm forward of the wheel axis (base_link
+       origin). depth_camera_x is chassis-local (this macro's parent_link
+       is "chassis", whose own origin sits at chassis_joint_x relative to
+       base_link — see mserve_core.xacro), so it's the wheel-axis-relative
+       measurement minus chassis_joint_x. -->
+  <xacro:property name="depth_camera_x_from_wheel_axis" value="0.280"/>
+  <xacro:property name="depth_camera_x" value="${depth_camera_x_from_wheel_axis - chassis_joint_x}"/>
   <xacro:property name="depth_camera_y" value="0.0"/>
+  <!-- Height above the wheel axis NOT yet updated — 115mm measured, but
+       chassis_height (still an unmeasured 150mm placeholder) alone already
+       exceeds that: chassis_height + depth_camera_height/2 as currently
+       written can't produce 115mm without chassis_height actually being
+       ~102mm, i.e. this depends on a real chassis_height measurement, not
+       just this camera's own numbers. Get that before touching this. -->
   <xacro:property name="depth_camera_z" value="${chassis_height + depth_camera_height / 2.0}"/>
   <xacro:property name="depth_camera_image_topic"   value="camera/image_raw"/>

File: ws/src/mserve_description/urdf/mserve_lidar.xacro (robot description, xacro)
@@ -1,15 +1,32 @@
 <?xml version="1.0"?>
 <robot xmlns:xacro="http://www.ros.org/wiki/xacro">
-  <!-- RPLIDAR C1 envelope and scan characteristics -->
-  <xacro:property name="lidar_radius" value="0.04"/>
-  <xacro:property name="lidar_length" value="0.04"/>
+  <!-- RPLIDAR C1 envelope and scan characteristics — measured 2026-07-19:
+       55x55x35mm (wxdxh). Approximated as a cylinder (radius = min(w,d)/2,
+       length = h) rather than switching to a box — close enough for a
+       collision/visual placeholder, and keeps the riser-stacking math
+       below simple. -->
+  <xacro:property name="lidar_radius" value="0.0275"/>
+  <xacro:property name="lidar_length" value="0.035"/>
   <xacro:property name="lidar_mass" value="0.11"/>
   <xacro:property name="lidar_riser_radius" value="0.012"/>
-  <xacro:property name="lidar_riser_height" value="0.06"/>
+  <!-- Measured 2026-07-19: 75mm forward of the wheel axis (base_link
+       origin). lidar_x is chassis-local (this macro's parent_link is
+       "chassis", whose own origin sits at chassis_joint_x relative to
+       base_link — see mserve_core.xacro), so it's the wheel-axis-relative
+       measurement minus chassis_joint_x (a negative number), not the
+       measurement directly. -->
+  <xacro:property name="lidar_x_from_wheel_axis" value="0.075"/>
+  <xacro:property name="lidar_x" value="${lidar_x_from_wheel_axis - chassis_joint_x}"/>
+  <xacro:property name="lidar_y" value="0.0"/>
   <xacro:property name="lidar_riser_mass" value="0.03"/>
-  <xacro:property name="lidar_offset" value="0.00"/>
-  <xacro:property name="lidar_x" value="${chassis_length / 2.0 + lidar_offset}"/>
-  <xacro:property name="lidar_y" value="0.0"/>
-  <xacro:property name="lidar_riser_z" value="${chassis_height + lidar_riser_height / 2.0}"/>
+  <!-- Height above the wheel axis (base_link) measured 2026-07-19: 175mm —
+       taken directly from the wheel axis per that measurement (no chassis
+       box in between; the real chassis is an open rail frame, not a solid
+       box — see mserve_core.xacro's chassis_joint_x comment), so
+       lidar_riser_z no longer goes through chassis_height. riser_height is
+       solved backwards from the 175mm target (riser_height + lidar_length/2
+       = 175mm) rather than being its own independent measurement. -->
+  <xacro:property name="lidar_riser_height" value="${0.175 - lidar_length / 2.0}"/>
+  <xacro:property name="lidar_riser_z" value="${lidar_riser_height / 2.0}"/>
   <xacro:property name="lidar_z" value="${lidar_riser_height / 2.0 + lidar_length / 2.0}"/>
   <xacro:property name="lidar_scan_topic" value="scan"/>
